File: PCB/PCB.sch (KiCad schematic (older format))
At the start: 52 parts, among them J1 Conn_01x03, J2 Conn_01x02, Q1 2N2907, Q10 TIP32, Q11 BD138, Q12 TIP31, Q13 2N2222, Q2 2N2907, Q3 2N2907, Q4 2N2222, Q5 2N2222, Q6 2N2907, Q7 2N2907, Q8 BD139, Q9 BD139, U11 Relai, U2 Jack_Mono

Commit message: Empreinte terminée, demander vérifs
Parts:
- C8: footprint (none) -> CmpAmpliAudio:C_Rect_L7.2mm_W3.5mm_P5.00mm_FKS2_FKP2_MKS2_MKP2
- R1, R10, R13, R14, R15, R16, R17, R2, R3, R4, R5, R6, R7, R8, R9: footprint (none) -> CmpAmpliAudio:R_Axial_DIN0207_L6.3mm_D2.5mm_P10.16mm_Horizontal
- R11, R12: footprint (none) -> CmpAmpliAudio:R_Axial_DIN0516_L15.5mm_D5.0mm_P20.32mm_Horizontal
- U11: footprint (none) -> CmpRelai:Relai
Changed lines of the file:
@@
 F 0 "R5" H 2470 2546 50  0000 L CNN
 F 1 "R" H 2470 2455 50  0000 L CNN
-F 2 "" V 2330 2500 50  0001 C CNN
+F 2 "CmpAmpliAudio:R_Axial_DIN0207_L6.3mm_D2.5mm_P10.16mm_Horizontal" V 2330 2500 50  0001 C CNN
 F 3 "~" H 2400 2500 50  0001 C CNN
 	1    2400 2500
@@
 F 0 "R1" H 2070 3796 50  0000 L CNN
 F 1 "R" H 2070 3705 50  0000 L CNN
-F 2 "" V 1930 3750 50  0001 C CNN
+F 2 "CmpAmpliAudio:R_Axial_DIN0207_L6.3mm_D2.5mm_P10.16mm_Horizontal" V 1930 3750 50  0001 C CNN
 F 3 "~" H 2000 3750 50  0001 C CNN
 	1    2000 3750
@@
 F 0 "R2" H 2770 4546 50  0000 L CNN
 F 1 "R" H 2770 4455 50  0000 L CNN
-F 2 "" V 2630 4500 50  0001 C CNN
+F 2 "CmpAmpliAudio:R_Axial_DIN0207_L6.3mm_D2.5mm_P10.16mm_Horizontal" V 2630 4500 50  0001 C CNN
 F 3 "~" H 2700 4500 50  0001 C CNN
 	1    2700 4500
@@
 F 0 "R15" H 4020 6146 50  0000 L CNN
 F 1 "R" H 4020 6055 50  0000 L CNN
-F 2 "" V 3880 6100 50  0001 C CNN
+F 2 "CmpAmpliAudio:R_Axial_DIN0207_L6.3mm_D2.5mm_P10.16mm_Horizontal" V 3880 6100 50  0001 C CNN
 F 3 "~" H 3950 6100 50  0001 C CNN
 	1    3950 6100
@@
 F 0 "R14" V 4850 5750 50  0000 L CNN
 F 1 "R" V 4750 5850 50  0000 L CNN
-F 2 "" V 4580 5800 50  0001 C CNN
+F 2 "CmpAmpliAudio:R_Axial_DIN0207_L6.3mm_D2.5mm_P10.16mm_Horizontal" V 4580 5800 50  0001 C CNN
 F 3 "~" H 4650 5800 50  0001 C CNN
 	1    4650 5800
@@
 F 0 "R4" H 3120 1546 50  0000 L CNN
 F 1 "R" H 3120 1455 50  0000 L CNN
-F 2 "" V 2980 1500 50  0001 C CNN
+F 2 "CmpAmpliAudio:R_Axial_DIN0207_L6.3mm_D2.5mm_P10.16mm_Horizontal" V 2980 1500 50  0001 C CNN
 F 3 "~" H 3050 1500 50  0001 C CNN
 	1    3050 1500
@@
 F 0 "R7" H 5320 1446 50  0000 L CNN
 F 1 "R" H 5320 1355 50  0000 L CNN
-F 2 "" V 5180 1400 50  0001 C CNN
+F 2 "CmpAmpliAudio:R_Axial_DIN0207_L6.3mm_D2.5mm_P10.16mm_Horizontal" V 5180 1400 50  0001 C CNN
 F 3 "~" H 5250 1400 50  0001 C CNN
 	1    5250 1400
@@
 F 0 "R9" H 4320 1446 50  0000 L CNN
 F 1 "R" H 4320 1355 50  0000 L CNN
-F 2 "" V 4180 1400 50  0001 C CNN
+F 2 "CmpAmpliAudio:R_Axial_DIN0207_L6.3mm_D2.5mm_P10.16mm_Horizontal" V 4180 1400 50  0001 C CNN
 F 3 "~" H 4250 1400 50  0001 C CNN
 	1    4250 1400
@@
 F 0 "R8" V 5150 3100 50  0000 L CNN
 F 1 "R" V 5050 3150 50  0000 L CNN
-F 2 "" V 4880 3150 50  0001 C CNN
+F 2 "CmpAmpliAudio:R_Axial_DIN0207_L6.3mm_D2.5mm_P10.16mm_Horizontal" V 4880 3150 50  0001 C CNN
 F 3 "~" H 4950 3150 50  0001 C CNN
 	1    4950 3150
@@
 F 0 "R3" H 3670 4546 50  0000 L CNN
 F 1 "R" H 3670 4455 50  0000 L CNN
-F 2 "" V 3530 4500 50  0001 C CNN
+F 2 "CmpAmpliAudio:R_Axial_DIN0207_L6.3mm_D2.5mm_P10.16mm_Horizontal" V 3530 4500 50  0001 C CNN
 F 3 "~" H 3600 4500 50  0001 C CNN
 	1    3600 4500
@@
 F 0 "R6" H 5320 4946 50  0000 L CNN
 F 1 "R" H 5320 4855 50  0000 L CNN
-F 2 "" V 5180 4900 50  0001 C CNN
+F 2 "CmpAmpliAudio:R_Axial_DIN0207_L6.3mm_D2.5mm_P10.16mm_Horizontal" V 5180 4900 50  0001 C CNN
 F 3 "~" H 5250 4900 50  0001 C CNN
 	1    5250 4900
@@
 F 0 "R11" H 6770 2846 50  0000 L CNN
 F 1 "R" H 6770 2755 50  0000 L CNN
-F 2 "" V 6630 2800 50  0001 C CNN
+F 2 "CmpAmpliAudio:R_Axial_DIN0516_L15.5mm_D5.0mm_P20.32mm_Horizontal" V 6630 2800 50  0001 C CNN
 F 3 "~" H 6700 2800 50  0001 C CNN
 	1    6700 2800
@@
 F 0 "R12" H 6770 3296 50  0000 L CNN
 F 1 "R" H 6770 3205 50  0000 L CNN
-F 2 "" V 6630 3250 50  0001 C CNN
+F 2 "CmpAmpliAudio:R_Axial_DIN0516_L15.5mm_D5.0mm_P20.32mm_Horizontal" V 6630 3250 50  0001 C CNN
 F 3 "~" H 6700 3250 50  0001 C CNN
 	1    6700 3250
@@
 F 0 "C8" H 8150 1600 50  0000 C CNN
 F 1 "470u" H 8200 1500 50  0000 C CNN
-F 2 "" H 8038 1400 50  0001 C CNN
+F 2 "CmpAmpliAudio:C_Rect_L7.2mm_W3.5mm_P5.00mm_FKS2_FKP2_MKS2_MKP2" H 8038 1400 50  0001 C CNN
 F 3 "~" H 8000 1550 50  0001 C CNN
 	1    8000 1550
@@
 F 0 "R13" H 7920 3396 50  0000 L CNN
 F 1 "R" H 7920 3305 50  0000 L CNN
-F 2 "" V 7780 3350 50  0001 C CNN
+F 2 "CmpAmpliAudio:R_Axial_DIN0207_L6.3mm_D2.5mm_P10.16mm_Horizontal" V 7780 3350 50  0001 C CNN
 F 3 "~" H 7850 3350 50  0001 C CNN
 	1    7850 3350
@@
 F 0 "R16" H 10070 4446 50  0000 L CNN
 F 1 "R" H 10070 4355 50  0000 L CNN
-F 2 "" V 9930 4400 50  0001 C CNN
+F 2 "CmpAmpliAudio:R_Axial_DIN0207_L6.3mm_D2.5mm_P10.16mm_Horizontal" V 9930 4400 50  0001 C CNN
 F 3 "~" H 10000 4400 50  0001 C CNN
 	1    10000 4400
@@
 F 0 "R17" H 9470 5346 50  0000 L CNN
 F 1 "R" H 9470 5255 50  0000 L CNN
-F 2 "" V 9330 5300 50  0001 C CNN
+F 2 "CmpAmpliAudio:R_Axial_DIN0207_L6.3mm_D2.5mm_P10.16mm_Horizontal" V 9330 5300 50  0001 C CNN
 F 3 "~" H 9400 5300 50  0001 C CNN
 	1    9400 5300
@@
 F 0 "R10" H 4320 2446 50  0000 L CNN
 F 1 "R" H 4320 2355 50  0000 L CNN
-F 2 "" V 4180 2400 50  0001 C CNN
+F 2 "CmpAmpliAudio:R_Axial_DIN0207_L6.3mm_D2.5mm_P10.16mm_Horizontal" V 4180 2400 50  0001 C CNN
 F 3 "~" H 4250 2400 50  0001 C CNN
 	1    4250 2400
@@
 F 0 "U11" H 9600 3517 50  0000 C CNN
 F 1 "Relai" H 9600 3426 50  0000 C CNN
-F 2 "" V 9250 3000 50  0001 C CNN
+F 2 "CmpRelai:Relai" V 9250 3000 50  0001 C CNN
 F 3 "" V 9250 3000 50  0001 C CNN
 	1    9650 3150

Commit message: on passe au routage
Parts:
- C4, C6: footprint (none) -> CmpAmpliAudio:CP_Radial_D8.0mm_P5.00mm
- RV1, RV2: footprint (none) -> CmpAmpliAudio:Potentiometer_Bourns_3296W_Vertical
Changed lines of the file:
@@
 encoding utf-8
 Sheet 1 1
-Title ""
-Date ""
-Rev ""
-Comp ""
+Title "PCB BE Elec"
+Date "2021-04-17"
+Rev "V0"
+Comp "INSA GEI"
 Comment1 ""
 Comment2 ""
@@
 F 0 "RV1" H 4600 2900 50  0000 R CNN
 F 1 "R_POT" H 4650 2800 50  0000 R CNN
-F 2 "" H 4700 2800 50  0001 C CNN
+F 2 "CmpAmpliAudio:Potentiometer_Bourns_3296W_Vertical" H 4700 2800 50  0001 C CNN
 F 3 "~" H 4700 2800 50  0001 C CNN
 	1    4700 2800
@@
 F 0 "C6" H 2550 6900 50  0000 C CNN
 F 1 "10u" H 2550 6800 50  0000 C CNN
-F 2 "" H 2388 6700 50  0001 C CNN
+F 2 "CmpAmpliAudio:CP_Radial_D8.0mm_P5.00mm" H 2388 6700 50  0001 C CNN
 F 3 "~" H 2350 6850 50  0001 C CNN
 	1    2350 6850
@@
 F 0 "C4" H 2550 6300 50  0000 C CNN
 F 1 "10u" H 2550 6200 50  0000 C CNN
-F 2 "" H 2388 6100 50  0001 C CNN
+F 2 "CmpAmpliAudio:CP_Radial_D8.0mm_P5.00mm" H 2388 6100 50  0001 C CNN
 F 3 "~" H 2350 6250 50  0001 C CNN
 	1    2350 6250
@@
 F 0 "RV2" H 4650 3000 50  0000 R CNN
 F 1 "R_POT" H 4750 2900 50  0000 R CNN
-F 2 "" H 4250 2850 50  0001 C CNN
+F 2 "CmpAmpliAudio:Potentiometer_Bourns_3296W_Vertical" H 4250 2850 50  0001 C CNN
 F 3 "~" H 4250 2850 50  0001 C CNN
 	1    4250 2850

Commit message: tout est placé mais il faut réorganiser
Parts:
- removed C8: 470u, CmpAmpliAudio:C_Rect_L7.2mm_W3.5mm_P5.00mm_FKS2_FKP2_MKS2_MKP2, symbol Device:C
- added C8: 470u, CmpAmpliAudio:CP_Radial_D12.5mm_P5.00mm, symbol Device:CP
Connections:
- net +12V: now also C8.1
- net GND: now also C8.2
Changed lines of the file:
@@
-$EndComp
-$Comp
-L Device:C C8
-U 1 1 605DC49D
-P 8000 1550
-F 0 "C8" H 8150 1600 50  0000 C CNN
-F 1 "470u" H 8200 1500 50  0000 C CNN
-F 2 "CmpAmpliAudio:C_Rect_L7.2mm_W3.5mm_P5.00mm_FKS2_FKP2_MKS2_MKP2" H 8038 1400 50  0001 C CNN
-F 3 "~" H 8000 1550 50  0001 C CNN
-	1    8000 1550
-	1    0    0    -1
 $EndComp
 $Comp
@@
 	1    0    0    -1
 $EndComp
+$Comp
+L Device:CP C8
+U 1 1 606F65FC
+P 8000 1550
+F 0 "C8" H 8150 1650 50  0000 C CNN
+F 1 "470u" H 8200 1550 50  0000 C CNN
+F 2 "CmpAmpliAudio:CP_Radial_D12.5mm_P5.00mm" H 8038 1400 50  0001 C CNN
+F 3 "~" H 8000 1550 50  0001 C CNN
+	1    8000 1550
+	1    0    0    -1
+$EndComp
