File: PCB/PCB.kicad_pcb (KiCad board)
At the start: 2 copper layers, 110 x 100 mm, 52 parts, among them J1 Conn_01x03, J2 Conn_01x02, Q1 2N2907, Q10 TIP32, Q11 BD138, Q12 TIP31, Q13 2N2222, Q2 2N2907, Q3 2N2907, Q4 2N2222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

Commit message: placement ok !
Parts:
- moved Q12 5.68 mm to (133.3, 77.5), turned to 180 degrees
- moved Q8 1.27 mm to (128.3, 85.1)
Other:
- net class Default: via_dia 1.9 -> 2.1
Changed lines of the file:
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@@
     (zone_45_only no)
     (trace_min 0.4)
-    (via_size 1.9)
+    (via_size 2.1)
     (via_drill 0.6)
     (via_min_size 0.6)
     (via_min_drill 0.6)
-    (user_via 1.9 0.6)
+    (user_via 2.1 0.6)
     (uvia_size 1)
     (uvia_drill 0.6)
@@
     (pad_to_mask_clearance 0)
     (aux_axis_origin 0 0)
-    (visible_elements 7FFFFFFF)
+    (visible_elements 7FFFF7FF)
     (pcbplotparams
       (layerselection 0x010fc_ffffffff)
@@
     (clearance 0.3)
     (trace_width 0.6)
-    (via_dia 1.9)
+    (via_dia 2.1)
     (via_drill 0.6)
     (uvia_dia 1)
@@
   )
   (module CmpAmpliAudio:TO-220-3_Vertical (layer F.Cu)
-    (at 128.27 80.01)
+    (at 133.35 77.47 180)
     (descr "TO-220-3, Vertical, RM 2.54mm, see https://www.vishay.com/docs/66542/to-220-1.pdf")
     (tags "TO-220-3 Vertical RM 2.54mm")
@@
       (effects (font (size 1 1) (thickness 0.15)))
     )
-    (pad 1 thru_hole rect (at 0 0) (size 1.8 2.7) (drill 1.1) (layers *.Cu *.Mask)
+    (pad 1 thru_hole rect (at 0 0 180) (size 1.8 2.7) (drill 1.1) (layers *.Cu *.Mask)
       (net 27 "Net-(Q11-Pad2)"))
-    (pad 2 thru_hole rect (at 2.54 0) (size 1.8 2.7) (drill 1.1) (layers *.Cu *.Mask)
+    (pad 2 thru_hole rect (at 2.54 0 180) (size 1.8 2.7) (drill 1.1) (layers *.Cu *.Mask)
       (net 26 "Net-(Q11-Pad1)"))
-    (pad 3 thru_hole rect (at 5.08 0) (size 1.8 2.7) (drill 1.1) (layers *.Cu *.Mask)
+    (pad 3 thru_hole rect (at 5.08 0 180) (size 1.8 2.7) (drill 1.1) (layers *.Cu *.Mask)
       (net 6 -12V))
     (model ${KISYS3DMOD}/Package_TO_SOT_THT.3dshapes/TO-220-3_Vertical.wrl
@@
   )
   (module CmpAmpliAudio:TO-126-3_Vertical (layer F.Cu)
-    (at 128.27 86.36)
+    (at 128.27 85.09)
     (descr "TO-126-3, Vertical, RM 2.54mm, see https://www.diodes.com/assets/Package-Files/TO126.pdf")
     (tags "TO-126-3 Vertical RM 2.54mm")

Commit message: 1er routage pas top
Parts:
- added D3: 1N4001, Diode_THT:D_DO-41_SOD81_P10.16mm_Horizontal, F.Cu at (118.1, 146.1)
- added D4: 1N4001, Diode_THT:D_DO-41_SOD81_P10.16mm_Horizontal, F.Cu at (147.3, 139.7)
- moved R9 3.81 mm to (118.1, 137.2)
- moved R7 2.54 mm to (111.8, 134.6)
Connections:
- J1 pad 1: -12V -> +12V
- J1 pad 3: +12V -> -12V
- J2 pad 1: GND -> Net-(J2-Pad1)
- J2 pad 2: Net-(J2-Pad1) -> GND
Routing:
- net GND: track 0.00 -> 368.4 mm
- net -12V: track 0.00 -> 286.3 mm
- net +12V: track 0.00 -> 176.4 mm
- net Net-(Q6-Pad3): track 0.00 -> 148.3 mm
- net Net-(R11-Pad2): track 0.00 -> 113.3 mm
- net Net-(C2-Pad1): track 0.00 -> 53.0 mm
- net Net-(Q10-Pad2): track 0.00 -> 42.1 mm
- net Net-(C3-Pad1): track 0.00 -> 38.4 mm
- net Net-(C1-Pad1): track 0.00 -> 33.1 mm
- net Net-(Q6-Pad2): track 0.00 -> 32.2 mm
- net Net-(Q11-Pad1): track 0.00 -> 31.7 mm
- net Net-(C2-Pad2): track 0.00 -> 25.6 mm
- net Net-(Q10-Pad1): track 0.00 -> 25.0 mm
- net Net-(Q11-Pad2): track 0.00 -> 23.5 mm
- net Net-(Q8-Pad3): track 0.00 -> 20.1 mm
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
Commit message: routage debut mieux
Routing:
- net Net-(Q6-Pad3): track 148.3 -> 20.1 mm
- net Net-(R11-Pad2): track 113.3 -> 7.93 mm
- net -12V: track 286.3 -> 184.2 mm
- net GND: track 368.4 -> 291.1 mm
- net +12V: track 176.4 -> 100.2 mm
- net Net-(C1-Pad1): track 33.1 -> 0.00 mm
- net Net-(Q6-Pad2): track 32.2 -> 0.00 mm
- net Net-(C3-Pad1): track 38.4 -> 7.62 mm
- net Net-(C2-Pad2): track 25.6 -> 0.00 mm
- net Net-(Q4-Pad1): track 19.3 -> 0.00 mm
- net Net-(C2-Pad1): track 53.0 -> 33.7 mm
- net Net-(D2-Pad1): track 19.2 -> 0.00 mm
- net Net-(D1-Pad2): track 14.4 -> 0.00 mm
- net Net-(C1-Pad2): track 14.4 -> 0.00 mm
- net Net-(R10-Pad2): track 14.1 -> 0.00 mm
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
Commit message: routage j'espère que c'est ok
Parts:
- moved U11 0.96 mm to (92.7, 61.0)
Routing:
- net Net-(Q2-Pad2): track 0.00 -> 276.0 mm
- net -12V: track 184.2 -> 385.4 mm
- net +12V: track 100.2 -> 273.4 mm
- net GND: track 291.1 -> 417.6 mm
- net Net-(R11-Pad2): track 7.93 -> 117.7 mm
- net Net-(Q6-Pad3): track 20.1 -> 99.0 mm
- net Net-(C2-Pad1): track 33.7 -> 97.2 mm
- net Net-(C3-Pad1): track 7.62 -> 45.3 mm
- net Net-(C1-Pad1): track 0.00 -> 33.1 mm
- net Net-(Q6-Pad2): track 0.00 -> 31.8 mm
- net Net-(C2-Pad2): track 0.00 -> 26.7 mm
- net Net-(D2-Pad1): track 0.00 -> 21.2 mm
- net Net-(Q4-Pad1): track 0.00 -> 19.3 mm
- net Net-(D1-Pad2): track 0.00 -> 14.4 mm
- net Net-(C1-Pad2): track 0.00 -> 14.4 mm
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